Commit message: Added inertial macros for wheels and chassis

File: src/kabot_launcher/description/urdf/chassis.xacro (robot description, xacro)
@@ -1,4 +1,5 @@
 <?xml version="1.0"?>
 <robot xmlns:xacro="http://www.ros.org/wiki/xacro">
+  <xacro:include filename="inertial_macros.xacro"/>
   <xacro:include filename="materials.xacro"/>
   <xacro:property name="chassis_radius" value="0.06"/>
@@ -13,4 +14,12 @@
       <material name="white"/>
     </visual>
+    <collision>
+      <geometry>
+        <cylinder radius="${chassis_radius}" length="${chassis_height}"/>
+      </geometry>
+    </collision>
+    <xacro:inertial_cylinder mass="0.1" radius="${chassis_radius}" length="${chassis_height}">
+      <origin xyz="0 0 0" rpy="0 0 0"/>
+    </xacro:inertial_cylinder>
   </link>
   <joint name="footprint_joint" type="fixed">

File: src/kabot_launcher/description/urdf/wheel.xacro (robot description, xacro)
@@ -1,4 +1,5 @@
 <?xml version="1.0"?>
 <robot xmlns:xacro="http://www.ros.org/wiki/xacro">
+    <xacro:include filename="inertial_macros.xacro"/>
     <xacro:macro name="wheel" params="origin name parent joint_type='continuous' direction wheel_radius=0.035 wheel_height=0.005">
         <link name="${name}_link">
@@ -9,4 +10,17 @@
                 <material name="blue"/>
             </visual>
+            <collision>
+                <geometry>
+                    <cylinder radius="${wheel_radius}" length="${wheel_height}"/>
+                </geometry>
+            </collision>
+            <collision>
+                <geometry>
+                    <cylinder radius="${wheel_radius}" length="${wheel_height}"/>
+                </geometry>
+            </collision>
+            <xacro:inertial_cylinder mass="0.1" radius="${wheel_radius}" length="${wheel_height}">
+                <origin xyz="0 0 0" rpy="0 0 0"/>
+            </xacro:inertial_cylinder>
         </link>
         <joint name="${name}_joint" type="${joint_type}">

Commit message: Gazebo diff_drive_controller

File: src/kabot_launcher/description/urdf/chassis.xacro (robot description, xacro)
@@ -33,3 +33,6 @@
     <origin xyz="0.0 0.0 0.0"/>
   </joint>
+  <gazebo reference="chassis_link">
+    <material>Gazebo/Orange</material>
+  </gazebo>
 </robot>

File: src/kabot_launcher/description/urdf/kabot.urdf.xacro (robot description, xacro)
@@ -3,5 +3,6 @@
     <xacro:include filename="chassis.xacro"/>
     <xacro:include filename="wheel.xacro"/>
-    <xacro:wheel name="left_wheel" origin="0 ${chassis_radius-0.005} -0.005" parent="chassis_link" direction="1"/>
-    <xacro:wheel name="right_wheel" origin="0 -${chassis_radius-0.005} -0.005" parent="chassis_link" direction="-1"/>
+    <xacro:wheel name="left_wheel" origin="0 ${chassis_radius+0.005} -0.005" parent="chassis_link" direction="1"/>
+    <xacro:wheel name="right_wheel" origin="0 -${chassis_radius+0.005} -0.005" parent="chassis_link" direction="1"/>
+    <xacro:include filename="gazebo_control.xacro"/>
 </robot>

File: src/kabot_launcher/description/urdf/wheel.xacro (robot description, xacro)
@@ -30,4 +30,7 @@
             <axis xyz="0 0 ${direction}"/>
         </joint>
+        <gazebo reference="${name}_link">
+            <material>Gazebo/Blue</material>
+        </gazebo>
     </xacro:macro>
 </robot>
