Commit message: First small readme, additional launch files

File: src/kabot_launcher/description/urdf/wheel.xacro (robot description, xacro)
@@ -10,9 +10,4 @@
                 <material name="blue"/>
             </visual>
-            <collision>
-                <geometry>
-                    <cylinder radius="${wheel_radius}" length="${wheel_height}"/>
-                </geometry>
-            </collision>
             <collision>
                 <geometry>
